File: esp-led-dimmer.kicad_pcb (KiCad board)
At the start: 2 copper layers, 22.5 x 36.5 mm, 16 parts, among them J1 Barrel Jack 3A, J2 ESP-01, J3 LED 1, J4 LED 2, Q1 AO3400A, Q2 AO3400A, U1 TPS5430DDA

Commit message: Remove JLCPCB order marker placeholder
Other:
- board text removed: "JLCJLCJLCJLC"
Changed lines of the file:
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@@
-		)
-	)
-	(gr_text "JLCJLCJLCJLC"
-		(at 140.3 117.9 0)
-		(layer "F.SilkS")
-		(effects
-			(font
-				(size 0.8 0.8)
-				(thickness 0.1)
-			)
-			(justify left bottom)
 		)
 	)

Commit message: Replace screw terminal footprints
Parts:
- J3, J4: footprint TerminalBlock_Phoenix:TerminalBlock_Phoenix_MKDS-1,5-2_1x02_P5.00mm_Horizontal -> TerminalBlock:TerminalBlock_bornier-2_P5.08mm
- moved J4 1.65 mm to (142.1, 112.4)
- moved J3 1.65 mm to (153.4, 112.4)
Routing:
- net +24V: track 47.8 -> 45.3 mm
- net Net-(J4-Pin_1): track 7.60 -> 5.90 mm
- net Net-(J3-Pin_1): track 9.99 -> 9.41 mm
Other:
- board size 22.5 x 36.5 mm -> 22.5 x 33.5 mm
